Commit message: [1.01-1.02] Created ROS2 package

File: src/robot_urdf/urdf/robot_urdf.urdf.xacro (robot description, xacro)
@@ -1,3 +1,3 @@
-<?xml version="1.0" encoding="utf-8"?>
+<?xml version="1.0"?>
 <!-- This URDF was automatically created by SolidWorks to URDF Exporter! Originally created by Stephen Brawner (brawner@gmail.com)
      Commit Version: 1.6.0-4-g7f85cfe  Build Version: 1.6.7995.38578
@@ -5,4 +5,5 @@
 <robot name="robot_urdf" xmlns:xacro="http://www.ros.org/wiki/xacro">
   <xacro:include filename="$(find robot_urdf)/urdf/robot_urdf_gazebo.xacro"/>
+  <xacro:include filename="$(find robot_urdf)/urdf/robot_urdf_control.xacro"/>
   <!-- Dummy link to fix root inertia warning -->
   <link name="base_footprint"/>

File: src/robot_urdf/urdf/robot_urdf_gazebo.xacro (robot description, xacro)
@@ -1,10 +1,18 @@
 <?xml version="1.0" encoding="utf-8"?>
 <robot name="robot_urdf" xmlns:xacro="http://www.ros.org/wiki/xacro">
-  <!-- Gazebo plugin for ROS Control -->
-  <gazebo>
-    <plugin name="gazebo_ros_control" filename="libgazebo_ros_control.so">
-      <robotNamespace>/robot_urdf</robotNamespace>
-    </plugin>
-  </gazebo>
+  <transmission name="wheel_right_transmission">
+    <plugin>transmission_interface/SimpleTransmission</plugin>
+    <actuator name="wheel_right_motor" role="actuator_right"/>
+    <joint name="drive_wheel_joint_right" role="joint_right">
+      <mechanical_reduction>1.0</mechanical_reduction>
+    </joint>
+  </transmission>
+  <transmission name="wheel_left_transmission">
+    <plugin>transmission_interface/SimpleTransmission</plugin>
+    <actuator name="wheel_left_motor" role="actuator_left"/>
+    <joint name="drive_wheel_joint_left" role="joint_left">
+      <mechanical_reduction>1.0</mechanical_reduction>
+    </joint>
+  </transmission>
   <!-- Gazebo material and friction properties for links -->
   <gazebo reference="base_link">
@@ -71,21 +79,10 @@
     <minDepth>0.001</minDepth>
   </gazebo>
-  <!-- Gazebo plugin for Differential Drive -->
+  <!-- Gazebo plugin for ROS Control -->
   <gazebo>
-    <plugin name="differential_drive_controller" filename="libgazebo_ros_diff_drive.so">
-      <update_rate>50</update_rate>
-      <left_joint>drive_wheel_joint_left</left_joint>
-      <right_joint>drive_wheel_joint_right</right_joint>
-      <wheel_separation>0.21</wheel_separation>
-      <wheel_diameter>0.16</wheel_diameter>
-      <max_wheel_torque>20</max_wheel_torque>
-      <max_wheel_acceleration>1.0</max_wheel_acceleration>
-      <command_topic>cmd_vel</command_topic>
-      <publish_odom>true</publish_odom>
-      <publish_odom_tf>true</publish_odom_tf>
-      <publish_wheel_tf>false</publish_wheel_tf>
-      <odometry_topic>odom</odometry_topic>
-      <odometry_frame>odom</odometry_frame>
-      <robot_base_frame>base_footprint</robot_base_frame>
+    <plugin name="gazebo_ros2_control" filename="libgazebo_ros_control.so">
+      <robot_param>/robot_urdf</robot_param>
+      <robot_param_node>robot_state_publisher</robot_param_node>
+      <parameters>$(find robot_controller)/config/robot_controller.yaml</parameters>
     </plugin>
   </gazebo>

Commit message: [1.03-1.04] Created initial UML diagrams and header files

File: src/robot_urdf/urdf/robot_urdf.urdf.xacro (robot description, xacro)
@@ -1,9 +1,6 @@
 <?xml version="1.0"?>
-<!-- This URDF was automatically created by SolidWorks to URDF Exporter! Originally created by Stephen Brawner (brawner@gmail.com)
-     Commit Version: 1.6.0-4-g7f85cfe  Build Version: 1.6.7995.38578
-     For more information, please see http://wiki.ros.org/sw_urdf_exporter -->
 <robot name="robot_urdf" xmlns:xacro="http://www.ros.org/wiki/xacro">
-  <xacro:include filename="$(find robot_urdf)/urdf/robot_urdf_gazebo.xacro"/>
-  <xacro:include filename="$(find robot_urdf)/urdf/robot_urdf_control.xacro"/>
+  <xacro:include filename="$(find robot_urdf)/urdf/robot_urdf_gazebo.xacro" />
+  <xacro:include filename="$(find robot_urdf)/urdf/robot_urdf_control.xacro" />
   <!-- Dummy link to fix root inertia warning -->
   <link name="base_footprint"/>

File: src/robot_urdf/urdf/robot_urdf_control.xacro (robot description, xacro)
@@ -1,20 +1,22 @@
 <?xml version="1.0"?>
-<robot name="robot_urdf" xmlns:xacro="http://www.ros.org/wiki/xacro">
-    <ros2_control type="system" name="RobotSystem">
+<robot xmlns:xacro="http://www.ros.org/wiki/xacro" name="robot_urdf">
+    <ros2_control name="RobotSystem" type="system">
+        <!-- ros2_control Gazebo -->
         <hardware>
             <plugin>gazebo_ros2_control/GazeboSystem</plugin>
         </hardware>
-        <joint name="drive_wheel_joint_right">
+        <!-- ros2_control Common Interfaces -->
+        <joint name="drive_wheel_joint_left">
             <command_interface name="velocity">
-                <param name="min">-1</param>
-                <param name="max">1</param>
+                <param name="min">-10</param>
+                <param name="max">10</param>
             </command_interface>
             <state_interface name="position"/>
             <state_interface name="velocity"/>
         </joint>
-        <joint name="drive_wheel_joint_left">
+        <joint name="drive_wheel_joint_right">
             <command_interface name="velocity">
-                <param name="min">-1</param>
-                <param name="max">1</param>
+                <param name="min">-10</param>
+                <param name="max">10</param>
             </command_interface>
             <state_interface name="position"/>

File: src/robot_urdf/urdf/robot_urdf_gazebo.xacro (robot description, xacro)
@@ -1,8 +1,9 @@
 <?xml version="1.0" encoding="utf-8"?>
 <robot name="robot_urdf" xmlns:xacro="http://www.ros.org/wiki/xacro">
+  <!-- Move this one to ros2 control -->
   <transmission name="wheel_right_transmission">
     <plugin>transmission_interface/SimpleTransmission</plugin>
     <actuator name="wheel_right_motor" role="actuator_right"/>
-    <joint name="drive_wheel_joint_right" role="joint_right">
+    <joint name="drive_wheel_joint_right"    role="joint_right">
       <mechanical_reduction>1.0</mechanical_reduction>
     </joint>
@@ -11,5 +12,5 @@
     <plugin>transmission_interface/SimpleTransmission</plugin>
     <actuator name="wheel_left_motor" role="actuator_left"/>
-    <joint name="drive_wheel_joint_left" role="joint_left">
+    <joint name="drive_wheel_joint_left"    role="joint_left">
       <mechanical_reduction>1.0</mechanical_reduction>
     </joint>
@@ -81,7 +82,5 @@
   <!-- Gazebo plugin for ROS Control -->
   <gazebo>
-    <plugin name="gazebo_ros2_control" filename="libgazebo_ros_control.so">
-      <robot_param>/robot_urdf</robot_param>
-      <robot_param_node>robot_state_publisher</robot_param_node>
+    <plugin name="gazebo_ros2_control" filename="libgazebo_ros2_control.so">
       <parameters>$(find robot_controller)/config/robot_controller.yaml</parameters>
     </plugin>
